Commit message: rename package to UR3

File: phosphobot/resources/urdf/UR3/urdf/UR3_with_gripper.urdf (robot description, URDF)
Before this commit: robot ur3, 21 links, 20 joints
Links:
- link base_link: geometry collision mesh filename=package://UR3/meshes/ur3/collision/base.stl; visual mesh filename=package://UR3/meshes/ur3/visual/base.dae
- link forearm_link: geometry collision mesh filename=package://UR3/meshes/ur3/collision/forearm.stl; visual mesh filename=package://UR3/meshes/ur3/visual/forearm.dae
- link robotiq_85_adapter_link: geometry collision mesh filename=package://UR3/meshes/robotiq/collision/robotiq_85_gripper_a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; visual mesh filename=package://UR3/meshes/robotiq/visual/robotiq_85_gripper_adap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
- link robotiq_85_base_link: geometry collision mesh filename=package://UR3/meshes/robotiq/collision/robotiq_85_gripper_b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; visual mesh filename=package://UR3/meshes/robotiq/visual/robotiq_85_gripper_base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
- link robotiq_85_left_finger_link: geometry collision mesh filename=package://UR3/meshes/robotiq/collision/robotiq_85_gripper_j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; visual mesh filename=package://UR3/meshes/robotiq/visual/robotiq_85_gripper_join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
- link robotiq_85_left_finger_tip_link: geometry collision mesh filename=package://UR3/meshes/robotiq/collision/robotiq_85_gripper_j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; visual mesh filename=package://UR3/meshes/robotiq/visual/robotiq_85_gripper_join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
- link robotiq_85_left_inner_knuckle_link: geometry collision mesh filename=package://UR3/meshes/robotiq/collision/robotiq_85_gripper_j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; visual mesh filename=package://UR3/meshes/robotiq/visual/robotiq_85_gripper_join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
- link robotiq_85_left_knuckle_link: geometry collision mesh filename=package://UR3/meshes/robotiq/collision/robotiq_85_gripper_j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; visual mesh filename=package://UR3/meshes/robotiq/visual/robotiq_85_gripper_join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
- link robotiq_85_right_finger_link: geometry collision mesh filename=package://UR3/meshes/robotiq/collision/robotiq_85_gripper_j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; visual mesh filename=package://UR3/meshes/robotiq/visual/robotiq_85_gripper_join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
- link robotiq_85_right_finger_tip_link: geometry collision mesh filename=package://UR3/meshes/robotiq/collision/robotiq_85_gripper_j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; visual mesh filename=package://UR3/meshes/robotiq/visual/robotiq_85_gripper_join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
- link robotiq_85_right_inner_knuckle_link: geometry collision mesh filename=package://UR3/meshes/robotiq/collision/robotiq_85_gripper_j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; visual mesh filename=package://UR3/meshes/robotiq/visual/robotiq_85_gripper_join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
- link robotiq_85_right_knuckle_link: geometry collision mesh filename=package://UR3/meshes/robotiq/collision/robotiq_85_gripper_j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; visual mesh filename=package://UR3/meshes/robotiq/visual/robotiq_85_gripper_join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
- link shoulder_link: geometry collision mesh filename=package://UR3/meshes/ur3/collision/shoulder.stl; visual mesh filename=package://UR3/meshes/ur3/visual/shoulder.dae
- link upper_arm_link: geometry collision mesh filename=package://UR3/meshes/ur3/collision/upperarm.stl; visual mesh filename=package://UR3/meshes/ur3/visual/upperarm.dae
- link wrist_1_link: geometry collision mesh filename=package://UR3/meshes/ur3/collision/wrist1.stl; visual mesh filename=package://UR3/meshes/ur3/visual/wrist1.dae
- link wrist_2_link: geometry collision mesh filename=package://UR3/meshes/ur3/collision/wrist2.stl; visual mesh filename=package://UR3/meshes/ur3/visual/wrist2.dae
- link wrist_3_link: geometry collision mesh filename=package://UR3/meshes/ur3/collision/wrist3.stl; visual mesh filename=package://UR3/meshes/ur3/visual/wrist3.dae

Commit message: fixed dae error. recompiled dae to stl

File: phosphobot/resources/urdf/UR3/urdf/UR3_with_gripper.urdf (robot description, URDF)
Before this commit: robot ur3, 21 links, 20 joints
Links:
- link base_link: geometry collision mesh filename=meshes/ur3/collision/base.stl; visual mesh filename=meshes/ur3/visual/base.stl
- link forearm_link: geometry collision mesh filename=meshes/ur3/collision/forearm.stl; visual mesh filename=meshes/ur3/visual/forearm.stl
- link robotiq_85_adapter_link: geometry collision mesh filename=meshes/robotiq/collision/robotiq_85_gripper_adapter_plate.s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; visual mesh filename=meshes/robotiq/visual/robotiq_85_gripper_adapter_plate.stl
- link robotiq_85_base_link: geometry collision mesh filename=meshes/robotiq/collision/robotiq_85_gripper_base.stl; visual mesh filename=meshes/robotiq/visual/robotiq_85_gripper_base.stl
- link robotiq_85_left_finger_link: geometry collision mesh filename=meshes/robotiq/collision/robotiq_85_gripper_joint_1_L.stl; visual mesh filename=meshes/robotiq/visual/robotiq_85_gripper_joint_1_L.stl
- link robotiq_85_left_finger_tip_link: geometry collision mesh filename=meshes/robotiq/collision/robotiq_85_gripper_joint_3_L.stl; visual mesh filename=meshes/robotiq/visual/robotiq_85_gripper_joint_3_L.stl
- link robotiq_85_left_inner_knuckle_link: geometry collision mesh filename=meshes/robotiq/collision/robotiq_85_gripper_joint_2_L.stl; visual mesh filename=meshes/robotiq/visual/robotiq_85_gripper_joint_2_L.stl
- link robotiq_85_left_knuckle_link: geometry collision mesh filename=meshes/robotiq/collision/robotiq_85_gripper_joint_0_L.stl; visual mesh filename=meshes/robotiq/visual/robotiq_85_gripper_joint_0_L.stl
- link robotiq_85_right_finger_link: geometry collision mesh filename=meshes/robotiq/collision/robotiq_85_gripper_joint_1_R.stl; visual mesh filename=meshes/robotiq/visual/robotiq_85_gripper_joint_1_R.stl
- link robotiq_85_right_finger_tip_link: geometry collision mesh filename=meshes/robotiq/collision/robotiq_85_gripper_joint_3_R.stl; visual mesh filename=meshes/robotiq/visual/robotiq_85_gripper_joint_3_R.stl
- link robotiq_85_right_inner_knuckle_link: geometry collision mesh filename=meshes/robotiq/collision/robotiq_85_gripper_joint_2_R.stl; visual mesh filename=meshes/robotiq/visual/robotiq_85_gripper_joint_2_R.stl
- link robotiq_85_right_knuckle_link: geometry collision mesh filename=meshes/robotiq/collision/robotiq_85_gripper_joint_0_R.stl; visual mesh filename=meshes/robotiq/visual/robotiq_85_gripper_joint_0_R.stl
- link shoulder_link: geometry collision mesh filename=meshes/ur3/collision/shoulder.stl; visual mesh filename=meshes/ur3/visual/shoulder.stl
- link upper_arm_link: geometry collision mesh filename=meshes/ur3/collision/upperarm.stl; visual mesh filename=meshes/ur3/visual/upperarm.stl
- link wrist_1_link: geometry collision mesh filename=meshes/ur3/collision/wrist1.stl; visual mesh filename=meshes/ur3/visual/wrist1.stl
- link wrist_2_link: geometry collision mesh filename=meshes/ur3/collision/wrist2.stl; visual mesh filename=meshes/ur3/visual/wrist2.stl
- link wrist_3_link: geometry collision mesh filename=meshes/ur3/collision/wrist3.stl; visual mesh filename=meshes/ur3/visual/wrist3.stl

File: phosphobot/resources/urdf/UR3/urdf/robotiq_c2_model.urdf (robot description, URDF)
Before this commit: robot robotiq_c2_model, 11 links, 10 joints
Links:
- link robotiq_85_adapter_link: geometry collision mesh filename=meshes/robotiq/collision/robotiq_85_gripper_adapter_plate.s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; visual mesh filename=meshes/robotiq/visual/robotiq_85_gripper_adapter_plate.stl
- link robotiq_85_base_link: geometry collision mesh filename=meshes/robotiq/collision/robotiq_85_gripper_base.stl; visual mesh filename=meshes/robotiq/visual/robotiq_85_gripper_base.stl
- link robotiq_85_left_finger_link: geometry collision mesh filename=meshes/robotiq/collision/robotiq_85_gripper_joint_1_L.stl; visual mesh filename=meshes/robotiq/visual/robotiq_85_gripper_joint_1_L.stl
- link robotiq_85_left_finger_tip_link: geometry collision mesh filename=meshes/robotiq/collision/robotiq_85_gripper_joint_3_L.stl; visual mesh filename=meshes/robotiq/visual/robotiq_85_gripper_joint_3_L.stl
- link robotiq_85_left_inner_knuckle_link: geometry collision mesh filename=meshes/robotiq/collision/robotiq_85_gripper_joint_2_L.stl; visual mesh filename=meshes/robotiq/visual/robotiq_85_gripper_joint_2_L.stl
- link robotiq_85_left_knuckle_link: geometry collision mesh filename=meshes/robotiq/collision/robotiq_85_gripper_joint_0_L.stl; visual mesh filename=meshes/robotiq/visual/robotiq_85_gripper_joint_0_L.stl
- link robotiq_85_right_finger_link: geometry collision mesh filename=meshes/robotiq/collision/robotiq_85_gripper_joint_1_R.stl; visual mesh filename=meshes/robotiq/visual/robotiq_85_gripper_joint_1_R.stl
- link robotiq_85_right_finger_tip_link: geometry collision mesh filename=meshes/robotiq/collision/robotiq_85_gripper_joint_3_R.stl; visual mesh filename=meshes/robotiq/visual/robotiq_85_gripper_joint_3_R.stl
- link robotiq_85_right_inner_knuckle_link: geometry collision mesh filename=meshes/robotiq/collision/robotiq_85_gripper_joint_2_R.stl; visual mesh filename=meshes/robotiq/visual/robotiq_85_gripper_joint_2_R.stl
- link robotiq_85_right_knuckle_link: geometry collision mesh filename=meshes/robotiq/collision/robotiq_85_gripper_joint_0_R.stl; visual mesh filename=meshes/robotiq/visual/robotiq_85_gripper_joint_0_R.stl

File: phosphobot/resources/urdf/UR3/urdf/universalUR3.urdf (robot description, URDF)
Before this commit: robot ur3, 11 links, 10 joints
Links:
- link base_link: geometry collision mesh filename=meshes/ur3/collision/base.stl; visual mesh filename=meshes/ur3/visual/base.stl
- link forearm_link: geometry collision mesh filename=meshes/ur3/collision/forearm.stl; visual mesh filename=meshes/ur3/visual/forearm.stl
- link shoulder_link: geometry collision mesh filename=meshes/ur3/collision/shoulder.stl; visual mesh filename=meshes/ur3/visual/shoulder.stl
- link upper_arm_link: geometry collision mesh filename=meshes/ur3/collision/upperarm.stl; visual mesh filename=meshes/ur3/visual/upperarm.stl
- link wrist_1_link: geometry collision mesh filename=meshes/ur3/collision/wrist1.stl; visual mesh filename=meshes/ur3/visual/wrist1.stl
- link wrist_2_link: geometry collision mesh filename=meshes/ur3/collision/wrist2.stl; visual mesh filename=meshes/ur3/visual/wrist2.stl
- link wrist_3_link: geometry collision mesh filename=meshes/ur3/collision/wrist3.stl; visual mesh filename=meshes/ur3/visual/wrist3.stl
