Commit message: Changed the orientation of the gripper relative to the UR3

File: phosphobot/resources/urdf/UR3/urdf/UR3_with_gripper_bullet.urdf (robot description, URDF)
Before this commit: robot ur3, 19 links, 18 joints
Joints:
- joint mount_gripper_to_tool0: origin xyz=0 0 0 rpy=0 0 0 -> xyz=0 0 0 rpy=0 -1.55 0
